File: Hardware/SparkFun_Venus_GPS_SMA_Connector.brd (EAGLE design)
At the start: 29.2 x 17.8 mm, 31 parts, among them U1 VENUS638FLPX-L

Commit message: Updated PWR-RF GND jumper to fix Eagle issue
The Venus has power and rf grounds that should only connect at one place
on the board (R7). There was an issue with Eagle not automatically
connecting to this ground, leaving airwires. Part updated and overt
traces added.
Parts:
- moved R7 0.64 mm to (20.6, 12.1)
Routing:
- net RFGND: track 5.15 -> 6.58 mm
